File: teams/power/Battery Board/Battery Board V4/Battery board V4.1 - simple signals.brd (EAGLE design)
At the start: 90 x 90 mm, 54 parts, among them IC2 TPS77001

Commit message: Ongoing design changes in battery board V4.1
Parts:
- removed CIN1: 1uF, eagle-ltspice:C0805
- removed CIN2: 2.2uF, eagle-ltspice:C0805
- removed IC2: TPS77001, texas:SOT23-DBV
- removed R22: 5k, rcl:R0805
- removed SENSE1, SENSE2: 698, rcl:R0805
- removed U$6: LM57, Parts for Power Team:TSSOP-8
- added J1, J2, J3, J4: (no value), SparkFun-Connectors:1X02_LONGPADS
- added R15: 500k, rcl:R0805
- added R24, R25, R26, R27, R28: (no value), rcl:R0805
- added TP1, TP4: PTR1PAD1-13Y, testpad:P1-13Y
- added U$10: LM135Z, Parts for Power Team1:TO-92-3
- added VR1: 10k, SparkFun-Resistors:TRIMPOT-SMD-TC33X
- R13: value 10k -> 500k
- moved CIN7 117.2 mm to (67.8, 62.4)
- moved CIN6 106.0 mm to (60.3, 60.3), turned to 180 degrees
- moved CIN5 92.7 mm to (45.9, 60.3)
- moved CIN4 90.9 mm to (45.9, 64.5), turned to 180 degrees
- moved R14 85.3 mm to (45.9, 62.4)
- moved R13 38.1 mm to (67.8, 60.3), turned to 0 degrees
- moved R4 33.2 mm to (50.0, 39.6), turned to 180 degrees
- moved R5 30.9 mm to (57.1, 40.7), turned to 180 degrees
- moved RVD 27.8 mm to (47.5, 16.3), turned to 270 degrees
- moved R18 26.6 mm to (57.1, 38.4), turned to 180 degrees
- moved RLIM 24.0 mm to (50.0, 37.6), turned to 180 degrees
- moved CIN 22.9 mm to (45.9, 35.1), turned to 90 degrees
- moved R7 22.4 mm to (57.4, 17.3), turned to 270 degrees
- moved R19 22.4 mm to (57.2, 36.1), turned to 180 degrees
- moved C1 21.0 mm to (55.4, 17.7), turned to 90 degrees
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Connections:
- removed net 3.3V: CIN5.1, R14.1, U$7.P$54, U$7.P$55
- removed net CAN-5V: U$1.5V, U$7.P$50, U$7.P$51
- removed net LDO-5V: CIN2.1, IC2.5, R21.2, R4.2, U$6.4
- removed net N$13: U$6.7
- removed net TRIP-TEST: R22.2, U$6.5
- new net 3V3: CIN5.1, R14.1, U$1.3.3V@CAN1, U$1.3.3V@CAN2, U$1.3.3V@MSP1, U$1.3.3V@MSP2, U$7.P$54, U$7.P$55
- new net 5V: R21.2, R24.2, U$1.5V, U$7.P$50, U$7.P$51
- new net N$23: R24.1, R26.1, R27.2, TP1.TP, U$10.2, VR1.3
- new net N$24: R25.1, R26.2, TP4.TP, U$10.3, VR1.2
- new net N$3: J1.1, R5.1
- new net VOLTAGE-ADC_FILTERED: CIN6.1, R15.1, U$1.P1.1_A1
- new net VTEMP_FILTERED: CIN7.1, R13.1, U$1.P1.0_A0
- net ALCC: no longer U$7.P$41
- net GND: now also J1.2, J2.2, J3.2, J4.2, R25.2, R28.1, R4.1, U$10.1, VR1.1; no longer CIN1.2, CIN2.2, IC2.2, R13.1, R22.1, SENSE1.1, SENSE2.1, U$6.1
- net HEATER1: now also J3.1; no longer R18.1, R20.1, R5.1
- net IN-OUT: no longer CIN1.1, IC2.1
- net LDO-EN: no longer IC2.3, R13.2, U$7.P$34
- net N$11: now also J2.1, R18.1; no longer SENSE1.2, U$6.2
- net N$12: now also J4.1, R20.1; no longer SENSE2.2, U$6.3
- net OUT: no longer U$7.P$38
- net SCL: no longer U$7.P$33
- net SDA: no longer U$7.P$37
- net TOVER: now also R4.2; no longer R4.1, U$6.6
- net VOLTAGE-ADC: now also R15.2; no longer CIN6.1, U$1.P1.1_A1, U$7.P$42
- net VTEMP: now also R13.2, R27.1, R28.2; no longer CIN7.1, U$1.P1.0_A0, U$6.8, U$7.P$35
Routing:
- net VTEMP: track 151.7 -> 2.15 mm, vias 8 -> 0
- net LDO-EN: track 94.6 -> 0.00 mm, vias 8 -> 0
- net CAN-5V: track 89.0 -> 0.00 mm, vias 6 -> 0
- net CANL: track 89.0 -> 0.00 mm, vias 8 -> 0
- net CANH: track 88.4 -> 0.00 mm, vias 8 -> 0
- net OUT: track 80.8 -> 1.90 mm, vias 6 -> 2
- net VOLTAGE-ADC: track 81.9 -> 5.71 mm, vias 6 -> 0
- net 3.3V: track 74.3 -> 0.00 mm, vias 2 -> 0
- net TOVER: track 71.9 -> 5.90 mm, vias 7 -> 0
- net SCL: track 70.3 -> 6.96 mm, vias 6 -> 0
- net ALCC: track 74.4 -> 11.8 mm, vias 4 -> 0
- net SDA: track 65.3 -> 7.95 mm, vias 6 -> 0
- net SYNC1: track 55.6 -> 0.00 mm, vias 2 -> 0
- net SYNC2: track 54.7 -> 0.00 mm, vias 1 -> 0
- net GND: track 182.7 -> 129.0 mm
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