File: teams/power/Battery Board/Battery Board V4/Battery board V4.1 - simple signals.sch (EAGLE design)
At the start: 54 parts, among them IC2 TPS77001, Q1 TRANS_NPN-MMBT2222AL

Commit message: Ongoing design changes in battery board V4.1
Parts:
- removed CIN1: 1uF, eagle-ltspice:C
- removed CIN2: 2.2uF, eagle-ltspice:C
- removed IC2: TPS77001, texas:TPS77001
- removed R22: 5k, rcl:R-US_R0805
- removed SENSE1, SENSE2: 698, rcl:R-US_R0805
- removed U$6: LM57, Parts for Power Team:LM57
- added J1, J2, J3, J4: (no value), SparkFun-Connectors:CONN_02PTH3
- added R15: 500k, rcl:R-US_R0805
- added R24, R25, R26, R27, R28: (no value), rcl:R-US_R0805
- added TP1, TP4: PTR1PAD1-13Y, testpad:PTR1PAD1-13Y
- added U$10: LM135Z, Parts for Power Team1:LM135Z
- added VR1: 10k, SparkFun-Resistors:TRIMPOT-SMD-3MM-OPEN-1/10W-25%
- R13: value 10k -> 500k
Connections:
- removed net 3.3V: CIN5.1, R14.1, U$7.3.3V@54, U$7.3.3V@55
- removed net CAN-5V: U$1.5V_CAN, U$7.5V@50, U$7.5V@51
- removed net LDO-5V: CIN2.1, IC2.OUT, R21.2, R4.2, U$6.VDD
- removed net N$13: U$6.TOVER
- removed net TRIP-TEST: R22.2, U$6.TRIP-TEST
- new net 3V3: CIN5.1, R14.1, U$1.3.3V_CAN@1, U$1.3.3V_CAN@2, U$1.3.3V_MSP@2, U$1.3.3V_MSP@3, U$7.3.3V@54, U$7.3.3V@55
- new net 5V: R21.2, R24.2, U$1.5V_CAN, U$7.5V@50, U$7.5V@51
- new net N$23: R24.1, R26.1, R27.2, TP1.TP, U$10.P$+, VR1.CCW
- new net N$24: R25.1, R26.2, TP4.TP, U$10.P$ADJ, VR1.WIPER
- new net N$3: J1.1, R5.1
- new net VOLTAGE-ADC_FILTERED: CIN6.1, R15.1, U$1.P1.1_A1
- new net VTEMP_FILTERED: CIN7.1, R13.1, U$1.P1.0_A0
- net ALCC: no longer U$7.P$41
- net GND: now also J1.2, J2.2, J3.2, J4.2, R25.2, R28.1, R4.1, U$10.P$-, VR1.CW; no longer CIN1.2, CIN2.2, IC2.GND, R13.1, R22.1, SENSE1.1, SENSE2.1, U$6.GND
- net HEATER1: now also J3.1; no longer R18.1, R20.1, R5.1
- net IN-OUT: no longer CIN1.1, IC2.IN
- net LDO-EN: no longer IC2.!EN, R13.2, U$7.P$34
- net N$11: now also J2.1, R18.1; no longer SENSE1.2, U$6.SENSE1
- net N$12: now also J4.1, R20.1; no longer SENSE2.2, U$6.SENSE2
- net OUT: no longer U$7.P$38
- net SCL: no longer U$7.P$33
- net SDA: no longer U$7.P$37
- net TOVER: now also R4.2; no longer R4.1, U$6./TOVER/
- net VOLTAGE-ADC: now also R15.2; no longer CIN6.1, U$1.P1.1_A1, U$7.P$42
- net VTEMP: now also R13.2, R27.1, R28.2; no longer CIN7.1, U$1.P1.0_A0, U$6.VTEMP, U$7.P$35
Other:
- moved on the sheet: CIN7, R13, R4
