File: teams/power/Solar Panels/Center Panel V1/Center panel V1.2.brd (EAGLE design)
At the start: 82 x 277.8 mm, 7 parts

Commit message: Auto stash before merge of "develop" and "origin/develop"
Parts:
- removed J1: (no value), SparkFun-Connectors:1X05_1MM
- added U$7: PICOLOCK_5, DubSat1 Components:PICOLOCK_5
- moved U$4 5.00 mm to (40.9, 115.0), flipped to the bottom, turned to 270 degrees
- moved U$3 0.14 mm to (1.00, 88.0)
- moved U$1 0.11 mm to (1.00, 6.00)
- moved U$2 0.07 mm to (1.00, 47.0)
- moved U$5 0.05 mm to (1.00, 129.0)
Connections:
- removed net N$11: J1.3
- removed net N$12: J1.4
- removed net N$13: J1.5
- net GND: now also U$7.P$1; no longer J1.1
- net POWER: now also U$7.P$2; no longer J1.2
- net SCL: now also U$7.P$4
- net SDA: now also U$7.P$3
- net VS: now also U$7.P$5
Routing:
- net SDA: track 0.00 -> 10.8 mm
- net SCL: track 0.00 -> 9.26 mm
- net VS: track 0.00 -> 7.93 mm
- net GND: track 49.7 -> 51.9 mm
