File: teams/power/Solar Panels/Side Panel V1/side panel V5.brd (EAGLE design)
At the start: 82 x 277.8 mm, 7 parts

Commit message: Auto stash before merge of "develop" and "origin/develop"
Parts:
- removed J1: (no value), SparkFun-Connectors:1X05_LOCK
- added U$2, U$8: PICOLOCK_5, DubSat1 Components:PICOLOCK_5
- added U$9: INA219, DubSat1 Components:S008
Connections:
- new net SCL: U$2.P$2, U$8.P$4, U$9.5
- new net SDA: U$2.P$3, U$8.P$3, U$9.6
- new net VS: U$2.P$1, U$8.P$5, U$9.4
- net GND: now also U$2.P$5, U$8.P$1, U$9.3; no longer J1.1
- net POWER: now also U$2.P$4, U$8.P$2; no longer J1.2
Routing:
- net POWER: track 16.7 -> 136.9 mm, vias 0 -> 4
- net SDA: track 0.00 -> 42.6 mm
- net SCL: track 0.00 -> 40.7 mm
- net VS: track 0.00 -> 31.1 mm
- net GND: track 53.2 -> 56.8 mm
Changed lines of the file:
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@@
 <?xml version="1.0" encoding="utf-8"?>
 <!DOCTYPE eagle SYSTEM "eagle.dtd">
-<eagle version="7.6.0">
+<eagle version="8.3.1">
 <drawing>
 <settings>
 <setting alwaysvectorfont="no"/>
+<setting keepoldvectorfont="yes"/>
 <setting verticaltext="up"/>
 </settings>
@@
 </layers>
 <board>
+<fusionsync huburn="a.cGVyc29uYWw6dWUyOTMyNDU0" projecturn="a.cGVyc29uYWw6dWUyOTMyNDU0IzIwMTcwOTAxOTA3NDc1NTE" f3durn="urn:adsk.wipprod:dm.lineage:_qQpBSNdRFOLIfcIBuAhAg" pcbguid="2e365871-5002-4c73-93d4-943d870f15b6" lastpulledtime="" lastsyncedchangeguid="be041e69-810e-7fc2-1b29-6b85ead9e9e4"/>
 <plain>
 <wire x1="0" y1="268.67868125" x2="0" y2="277.8" width="0" layer="20"/>
@@
 </autorouter>
 <elements>
-<element name="U$3" library="DubSat1 Components" package="SOLAR_CELL_OUTLINE" value="SOALAR_CELL_OUTLINE" x="1" y="108"/>
-<element name="U$4" library="DubSat1 Components" package="SOLAR_CELL_OUTLINE" value="SOALAR_CELL_OUTLINE" x="1" y="149"/>
-<element name="U$5" library="DubSat1 Components" package="SOLAR_CELL_OUTLINE" value="SOALAR_CELL_OUTLINE" x="1" y="190"/>
-<element name="U$6" library="DubSat1 Components" package="SOLAR_CELL_TOP_SHORT-PAD" value="SOLAR_CELL_TOP" x="1" y="231"/>
-<element name="U$1" library="DubSat1 Components" package="SOLAR_CELL_STAND-ALONE" value="SOLAR_CELL_STAND-ALONE" x="1" y="8"/>
-<element name="U$7" library="DubSat1 Components" package="SOLAR_CELL_BOTTOM+BYPASS" value="SOLAR_CELL_BOTTOM+BYPASS" x="1" y="67"/>
-<element name="J1" library="SparkFun-Connectors" package="1X05_LOCK" value="" x="30.4" y="274"/>
+<element name="U$3" library="DubSat1 Components" library_urn="urn:adsk.eagle:library:348159" package="SOLAR_CELL_OUTLINE" package3d_urn="urn:adsk.eagle:package:348279/2" value="SOALAR_CELL_OUTLINE" x="1" y="108"/>
+<element name="U$4" library="DubSat1 Components" library_urn="urn:adsk.eagle:library:348159" package="SOLAR_CELL_OUTLINE" package3d_urn="urn:adsk.eagle:package:348279/2" value="SOALAR_CELL_OUTLINE" x="1" y="149"/>
+<element name="U$5" library="DubSat1 Components" library_urn="urn:adsk.eagle:library:348159" package="SOLAR_CELL_OUTLINE" package3d_urn="urn:adsk.eagle:package:348279/2" value="SOALAR_CELL_OUTLINE" x="1" y="190"/>
+<element name="U$6" library="DubSat1 Components" library_urn="urn:adsk.eagle:library:348159" package="SOLAR_CELL_TOP_SHORT-PAD" package3d_urn="urn:adsk.eagle:package:348280/2" value="SOLAR_CELL_TOP" x="1" y="231"/>
+<element name="U$1" library="DubSat1 Components" library_urn="urn:adsk.eagle:library:348159" package="SOLAR_CELL_STAND-ALONE" package3d_urn="urn:adsk.eagle:package:348283/2" value="SOLAR_CELL_STAND-ALONE" x="1" y="8"/>
+<element name="U$7" library="DubSat1 Components" library_urn="urn:adsk.eagle:library:348159" package="SOLAR_CELL_BOTTOM+BYPASS" package3d_urn="urn:adsk.eagle:package:348284/2" value="SOLAR_CELL_BOTTOM+BYPASS" x="1" y="67"/>
+<element name="U$2" library="DubSat1 Components" library_urn="urn:adsk.eagle:library:348159" package="PICOLOCK_5" package3d_urn="urn:adsk.eagle:package:348289/2" value="PICOLOCK_5" x="52" y="170" rot="MR90"/>
+<element name="U$8" library="DubSat1 Components" library_urn="urn:adsk.eagle:library:348159" package="PICOLOCK_5" package3d_urn="urn:adsk.eagle:package:348289/2" value="PICOLOCK_5" x="30" y="176" rot="MR270"/>
+<element name="U$9" library="DubSat1 Components" library_urn="urn:adsk.eagle:library:348159" package="S008" package3d_urn="urn:adsk.eagle:package:348285/2" value="INA219" x="41" y="160" rot="MR90"/>
 </elements>
 <signals>
@@
 <vertex x="82" y="0"/>
 </polygon>
-<contactref element="J1" pad="1"/>
 <contactref element="U$1" pad="P$1"/>
 <contactref element="U$1" pad="P$3"/>
@@
 <wire x1="61.5" y1="5.5" x2="61.9" y2="5.1" width="1.27" layer="1"/>
 <wire x1="61.9" y1="5.1" x2="67.5" y2="5.1" width="1.27" layer="1"/>
+<contactref element="U$9" pad="3"/>
+<contactref element="U$8" pad="P$1"/>
+<contactref element="U$2" pad="P$5"/>
+<wire x1="39.7" y1="160.325" x2="39.675" y2="160.35" width="0.2" layer="16"/>
+<wire x1="39.675" y1="160.35" x2="36.15" y2="160.35" width="0.2" layer="16"/>
 </signal>
 <signal name="N$9">
@@
 </signal>
 <signal name="POWER">
-<contactref element="J1" pad="2"/>
 <contactref element="U$6" pad="P$2"/>
-<wire x1="20.5" y1="273.5" x2="20.6" y2="273.6" width="1.27" layer="1"/>
-<wire x1="20.6" y1="273.6" x2="21.9" y2="273.6" width="1.27" layer="1"/>
-<wire x1="21.9" y1="273.6" x2="25.5" y2="270" width="1.27" layer="1"/>
-<wire x1="25.5" y1="270" x2="30.9" y2="270" width="1.27" layer="1"/>
-<wire x1="30.9" y1="270" x2="32.94" y2="272.04" width="1.27" layer="1"/>
-<wire x1="32.94" y1="272.04" x2="32.94" y2="273.873" width="1.27" layer="1"/>
+<contactref element="U$8" pad="P$2"/>
+<contactref element="U$2" pad="P$4"/>
+<via x="27.6" y="273.9" extent="1-16" drill="0.3"/>
+<via x="27.6" y="273.3" extent="1-16" drill="0.3"/>
+<via x="28.2" y="273.3" extent="1-16" drill="0.3"/>
+<via x="28.2" y="273.9" extent="1-16" drill="0.3"/>
+<wire x1="20.9" y1="273.9" x2="20.5" y2="273.5" width="1.016" layer="1"/>
+<wire x1="20.9" y1="273.9" x2="27.6" y2="273.9" width="1.016" layer="1"/>
+<wire x1="20.5" y1="273.5" x2="20.7" y2="273.3" width="1.016" layer="1"/>
+<wire x1="20.7" y1="273.3" x2="27.6" y2="273.3" width="1.016" layer="1"/>
+<wire x1="27.6" y1="273.3" x2="27.6" y2="175.8" width="1.016" layer="16"/>
+<wire x1="27.6" y1="175.8" x2="28.9" y2="174.5" width="0.6096" layer="16"/>
+<wire x1="28.9" y1="174.5" x2="30" y2="174.5" width="0.6096" layer="16"/>
+<wire x1="30" y1="174.5" x2="52" y2="174.5" width="0.6096" layer="16"/>
+<wire x1="28.2" y1="273.9" x2="28.2" y2="273.3" width="0" layer="19" extent="1-1"/>
+<wire x1="27.6" y1="273.3" x2="28.2" y2="273.3" width="0" layer="19" extent="16-16"/>
+</signal>
+<signal name="VS">
+<contactref element="U$9" pad="4"/>
+<contactref element="U$8" pad="P$5"/>
+<contactref element="U$2" pad="P$1"/>
+<wire x1="39.6308625" y1="170" x2="30" y2="170" width="0.2" layer="16"/>
+<wire x1="39.6308625" y1="170" x2="52" y2="170" width="0.2" layer="16"/>
+<wire x1="39.7" y1="160.975" x2="39.6308625" y2="161.0441375" width="0.2" layer="16"/>
+<wire x1="39.6308625" y1="161.0441375" x2="39.6308625" y2="170" width="0.2" layer="16"/>
+</signal>
+<signal name="SDA">
+<contactref element="U$9" pad="6"/>
+<contactref element="U$8" pad="P$3"/>
+<contactref element="U$2" pad="P$3"/>
+<wire x1="52" y1="173" x2="30" y2="173" width="0.2" layer="16"/>
+<wire x1="54.4032" y1="169.6329875" x2="54.4032" y2="171.0170125" width="0.2" layer="16"/>
+<wire x1="42.3" y1="160.325" x2="45.0952125" y2="160.325" width="0.2" layer="16"/>
+<wire x1="45.0952125" y1="160.325" x2="54.4032" y2="169.6329875" width="0.2" layer="16"/>
+<wire x1="52.4202125" y1="173" x2="52" y2="173" width="0.2" layer="16"/>
+<wire x1="54.4032" y1="171.0170125" x2="52.4202125" y2="173" width="0.2" layer="16"/>
+</signal>
+<signal name="SCL">
+<contactref element="U$9" pad="5"/>
+<contactref element="U$8" pad="P$4"/>
+<contactref element="U$2" pad="P$2"/>
+<wire x1="52" y1="171.5" x2="30" y2="171.5" width="0.2" layer="16"/>
+<wire x1="42.3" y1="160.975" x2="45.175" y2="160.975" width="0.2" layer="16"/>
+<wire x1="45.175" y1="160.975" x2="54" y2="169.8" width="0.2" layer="16"/>
+<wire x1="54" y1="169.8" x2="54" y2="170.85" width="0.2" layer="16"/>
+<wire x1="54" y1="170.85" x2="53.4" y2="171.45" width="0.2" layer="16"/>
+<wire x1="53.4" y1="171.45" x2="52.05" y2="171.45" width="0.2" layer="16"/>
+<wire x1="52.05" y1="171.45" x2="52" y2="171.5" width="0.2" layer="16"/>
 </signal>
 </signals>
 </board>
 </drawing>
+<compatibility>
+<note version="8.2" severity="warning">
+Since Version 8.2, EAGLE supports online libraries. The ids
+of those online libraries will not be understood (or retained)
+with this version.
+</note>
+<note version="8.3" severity="warning">
+Since Version 8.3, EAGLE supports Fusion synchronisation.
+This feature will not be available in this version and saving
+the document will break the link to the Fusion PCB feature.
+</note>
+<note version="8.3" severity="warning">
+Since Version 8.3, EAGLE supports URNs for individual library
+assets (packages, symbols, and devices). The URNs of those assets
+will not be understood (or retained) with this version.
+</note>
+<note version="8.3" severity="warning">
+Since Version 8.3, EAGLE supports the association of 3D packages
+with devices in libraries, schematics, and board files. Those 3D
+packages will not be understood (or retained) with this version.
+</note>
+</compatibility>
 </eagle>
