File: teams/power/Solar Panels/Side Panel V1/side panel V5.sch (EAGLE design)
At the start: 7 parts

Commit message: Auto stash before merge of "develop" and "origin/develop"
Parts:
- removed J1: (no value), SparkFun-Connectors:CONN_05LOCK
- added U$2, U$8: PICOLOCK_5, DubSat1 Components:PICOLOCK_5
- added U$9: INA219, DubSat1 Components:INA219
Connections:
- new net SCL: U$2.P$2, U$8.P$4, U$9.SCL
- new net SDA: U$2.P$3, U$8.P$3, U$9.SDA
- new net VS: U$2.P$1, U$8.P$5, U$9.VS
- net GND: now also U$2.P$5, U$8.P$1, U$9.GND; no longer J1.1
- net POWER: now also U$2.P$4, U$8.P$2; no longer J1.2
Changed lines of the file:
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@@
 <?xml version="1.0" encoding="utf-8"?>
 <!DOCTYPE eagle SYSTEM "eagle.dtd">
-<eagle version="7.6.0">
+<eagle version="8.3.1">
 <drawing>
 <settings>
 <setting alwaysvectorfont="no"/>
+<setting keepoldvectorfont="yes"/>
 <setting verticaltext="up"/>
 </settings>
@@
 </classes>
 <parts>
-<part name="U$3" library="DubSat1 Components" deviceset="SOALAR_CELL_OUTLINE" device=""/>
-<part name="U$4" library="DubSat1 Components" deviceset="SOALAR_CELL_OUTLINE" device=""/>
-<part name="U$5" library="DubSat1 Components" deviceset="SOALAR_CELL_OUTLINE" device=""/>
-<part name="U$6" library="DubSat1 Components" deviceset="SOLAR_CELL_TOP" device=""/>
-<part name="U$1" library="DubSat1 Components" deviceset="SOLAR_CELL_STAND-ALONE" device=""/>
-<part name="U$7" library="DubSat1 Components" deviceset="SOLAR_CELL_BOTTOM+BYPASS" device=""/>
-<part name="J1" library="SparkFun-Connectors" deviceset="CONN_05" device="LOCK"/>
+<part name="U$3" library="DubSat1 Components" library_urn="urn:adsk.eagle:library:348159" deviceset="SOALAR_CELL_OUTLINE" device="" package3d_urn="urn:adsk.eagle:package:348279/2"/>
+<part name="U$4" library="DubSat1 Components" library_urn="urn:adsk.eagle:library:348159" deviceset="SOALAR_CELL_OUTLINE" device="" package3d_urn="urn:adsk.eagle:package:348279/2"/>
+<part name="U$5" library="DubSat1 Components" library_urn="urn:adsk.eagle:library:348159" deviceset="SOALAR_CELL_OUTLINE" device="" package3d_urn="urn:adsk.eagle:package:348279/2"/>
+<part name="U$6" library="DubSat1 Components" library_urn="urn:adsk.eagle:library:348159" deviceset="SOLAR_CELL_TOP" device="" package3d_urn="urn:adsk.eagle:package:348280/2"/>
+<part name="U$1" library="DubSat1 Components" library_urn="urn:adsk.eagle:library:348159" deviceset="SOLAR_CELL_STAND-ALONE" device="" package3d_urn="urn:adsk.eagle:package:348283/2"/>
+<part name="U$7" library="DubSat1 Components" library_urn="urn:adsk.eagle:library:348159" deviceset="SOLAR_CELL_BOTTOM+BYPASS" device="" package3d_urn="urn:adsk.eagle:package:348284/2"/>
 <part name="GND1" library="SparkFun-PowerSymbols" deviceset="GND" device=""/>
+<part name="U$2" library="DubSat1 Components" library_urn="urn:adsk.eagle:library:348159" deviceset="PICOLOCK_5" device="" package3d_urn="urn:adsk.eagle:package:348289/2"/>
+<part name="U$8" library="DubSat1 Components" library_urn="urn:adsk.eagle:library:348159" deviceset="PICOLOCK_5" device="" package3d_urn="urn:adsk.eagle:package:348289/2"/>
+<part name="U$9" library="DubSat1 Components" library_urn="urn:adsk.eagle:library:348159" deviceset="INA219" device="" package3d_urn="urn:adsk.eagle:package:348285/2"/>
 </parts>
 <sheets>
@@
 <instance part="U$1" gate="G$1" x="2.54" y="-2.54"/>
 <instance part="U$7" gate="G$1" x="2.54" y="50.8"/>
-<instance part="J1" gate="G$1" x="81.28" y="251.46" rot="R180"/>
 <instance part="GND1" gate="1" x="35.56" y="-20.32"/>
+<instance part="U$2" gate="G$1" x="104.14" y="220.98" rot="R270"/>
+<instance part="U$8" gate="G$1" x="-33.02" y="223.52" rot="R90"/>
+<instance part="U$9" gate="G$1" x="109.22" y="167.64"/>
 </instances>
 <busses>
@@
 <net name="GND" class="0">
 <segment>
-<pinref part="J1" gate="G$1" pin="1"/>
-<wire x1="73.66" y1="256.54" x2="71.12" y2="256.54" width="0.1524" layer="91"/>
-<label x="68.58" y="256.54" size="1.778" layer="95"/>
-</segment>
-<segment>
 <pinref part="U$1" gate="G$1" pin="INTERCONNECTOR_1"/>
 <wire x1="15.24" y1="-7.62" x2="35.56" y2="-7.62" width="0.1524" layer="91"/>
@@
 <pinref part="U$1" gate="G$1" pin="INTERCONNECTOR_2"/>
 </segment>
+<segment>
+<pinref part="U$9" gate="G$1" pin="GND"/>
+<wire x1="96.52" y1="165.1" x2="88.9" y2="165.1" width="0.1524" layer="91"/>
+<label x="86.36" y="165.1" size="1.778" layer="95"/>
+</segment>
+<segment>
+<pinref part="U$8" gate="G$1" pin="P$1"/>
+<wire x1="-27.94" y1="210.82" x2="-20.32" y2="210.82" width="0.1524" layer="91"/>
+<label x="-20.32" y="210.82" size="1.778" layer="95"/>
+</segment>
+<segment>
+<pinref part="U$2" gate="G$1" pin="P$5"/>
+<wire x1="99.06" y1="213.36" x2="88.9" y2="213.36" width="0.1524" layer="91"/>
+<label x="86.36" y="213.36" size="1.778" layer="95"/>
+</segment>
 </net>
 <net name="POWER" class="0">
-<segment>
-<pinref part="J1" gate="G$1" pin="2"/>
-<wire x1="73.66" y1="254" x2="71.12" y2="254" width="0.1524" layer="91"/>
-<label x="66.04" y="254" size="1.778" layer="95"/>
-</segment>
 <segment>
 <pinref part="U$6" gate="G$1" pin="POSSITIVE_TAB"/>
 <wire x1="17.78" y1="251.46" x2="17.78" y2="256.54" width="0.1524" layer="91"/>
 <label x="15.24" y="256.54" size="1.778" layer="95"/>
+</segment>
+<segment>
+<pinref part="U$8" gate="G$1" pin="P$2"/>
+<wire x1="-27.94" y1="215.9" x2="-20.32" y2="215.9" width="0.1524" layer="91"/>
+<label x="-20.32" y="215.9" size="1.778" layer="95"/>
+</segment>
+<segment>
+<pinref part="U$2" gate="G$1" pin="P$4"/>
+<wire x1="99.06" y1="218.44" x2="88.9" y2="218.44" width="0.1524" layer="91"/>
+<label x="86.36" y="218.44" size="1.778" layer="95"/>
+</segment>
+</net>
+<net name="VS" class="0">
+<segment>
+<pinref part="U$9" gate="G$1" pin="VS"/>
+<wire x1="96.52" y1="160.02" x2="88.9" y2="160.02" width="0.1524" layer="91"/>
+<label x="86.36" y="160.02" size="1.778" layer="95"/>
+</segment>
+<segment>
+<pinref part="U$8" gate="G$1" pin="P$5"/>
+<wire x1="-27.94" y1="231.14" x2="-20.32" y2="231.14" width="0.1524" layer="91"/>
+<label x="-20.32" y="231.14" size="1.778" layer="95"/>
+</segment>
+<segment>
+<pinref part="U$2" gate="G$1" pin="P$1"/>
+<wire x1="99.06" y1="233.68" x2="88.9" y2="233.68" width="0.1524" layer="91"/>
+<label x="86.36" y="233.68" size="1.778" layer="95"/>
+</segment>
+</net>
+<net name="SDA" class="0">
+<segment>
+<pinref part="U$9" gate="G$1" pin="SDA"/>
+<wire x1="121.92" y1="165.1" x2="132.08" y2="165.1" width="0.1524" layer="91"/>
+<label x="129.54" y="165.1" size="1.778" layer="95"/>
+</segment>
+<segment>
+<pinref part="U$8" gate="G$1" pin="P$3"/>
+<wire x1="-27.94" y1="220.98" x2="-20.32" y2="220.98" width="0.1524" layer="91"/>
+<label x="-20.32" y="220.98" size="1.778" layer="95"/>
+</segment>
+<segment>
+<pinref part="U$2" gate="G$1" pin="P$3"/>
+<wire x1="99.06" y1="223.52" x2="88.9" y2="223.52" width="0.1524" layer="91"/>
+<label x="86.36" y="223.52" size="1.778" layer="95"/>
+</segment>
+</net>
+<net name="SCL" class="0">
+<segment>
+<pinref part="U$9" gate="G$1" pin="SCL"/>
+<wire x1="121.92" y1="160.02" x2="132.08" y2="160.02" width="0.1524" layer="91"/>
+<label x="129.54" y="160.02" size="1.778" layer="95"/>
+</segment>
+<segment>
+<pinref part="U$8" gate="G$1" pin="P$4"/>
+<wire x1="-27.94" y1="226.06" x2="-20.32" y2="226.06" width="0.1524" layer="91"/>
+<label x="-20.32" y="226.06" size="1.778" layer="95"/>
+</segment>
+<segment>
+<pinref part="U$2" gate="G$1" pin="P$2"/>
+<wire x1="99.06" y1="228.6" x2="88.9" y2="228.6" width="0.1524" layer="91"/>
+<label x="86.36" y="228.6" size="1.778" layer="95"/>
 </segment>
 </net>
@@
 </schematic>
 </drawing>
+<compatibility>
+<note version="8.2" severity="warning">
+Since Version 8.2, EAGLE supports online libraries. The ids
+of those online libraries will not be understood (or retained)
+with this version.
+</note>
+<note version="8.3" severity="warning">
+Since Version 8.3, EAGLE supports URNs for individual library
+assets (packages, symbols, and devices). The URNs of those assets
+will not be understood (or retained) with this version.
+</note>
+<note version="8.3" severity="warning">
+Since Version 8.3, EAGLE supports the association of 3D packages
+with devices in libraries, schematics, and board files. Those 3D
+packages will not be understood (or retained) with this version.
+</note>
+</compatibility>
 </eagle>
