File: teams/adcs/hardware/sensors/imu/LSM6DSM_breakout.brd (EAGLE design)
At the start: 20 x 27.5 mm, 6 parts

Commit message: ADCS/Sensors: Update eagle version in file header
Parts:
- C1, C2: value (none) -> 0.1 μF
Changed lines of the file:
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@@
 <?xml version="1.0" encoding="utf-8"?>
 <!DOCTYPE eagle SYSTEM "eagle.dtd">
-<eagle version="8.2.2">
+<eagle version="8.3.1">
 <drawing>
 <settings>
 <setting alwaysvectorfont="no"/>
+<setting keepoldvectorfont="yes"/>
 <setting verticaltext="up"/>
 </settings>
@@
 </autorouter>
 <elements>
-<element name="C1" library="rcl" library_urn="urn:adsk.eagle:library:334" package="C0805" value="" x="11.173" y="15.466" smashed="yes" rot="R90">
+<element name="C1" library="rcl" library_urn="urn:adsk.eagle:library:334" package="C0805" value="0.1 μF" x="11.173" y="15.466" smashed="yes" rot="R90">
 <attribute name="VALUE" x="13.713" y="14.196" size="1.27" layer="27" rot="R90"/>
 </element>
-<element name="C2" library="rcl" library_urn="urn:adsk.eagle:library:334" package="C0805" value="" x="10.14" y="7.16" smashed="yes" rot="R90">
+<element name="C2" library="rcl" library_urn="urn:adsk.eagle:library:334" package="C0805" value="0.1 μF" x="10.14" y="7.16" smashed="yes" rot="R90">
 <attribute name="VALUE" x="12.68" y="5.89" size="1.27" layer="27" rot="R90"/>
 </element>
@@
 <compatibility>
 <note version="8.2" severity="warning">
-Since Version 8.2, Eagle supports online libraries. The ids
+Since Version 8.2, EAGLE supports online libraries. The ids
 of those online libraries will not be understood (or retained)
 with this version.
