File: teams/power/Solar Panels/Side Panel V5/side panel V5.1.brd (EAGLE design)
At the start: 82 x 277.8 mm, 9 parts

Commit message: Tracking Side Panel V5.1 and V5.3, and moving Side Panel V5.x and associated files to it's own folder seperate from V4.
Parts:
- removed U$9: INA219, DubSat1 Components:S008
- added C3, C7: 100pF, Battery board V4.1 - simple signals:R0805
- added C4, C8: (no value), Battery board V4.1 - simple signals:C0805
- added U$10, U$12: TMP411, DubSat1 Components:TSSOP-8
- moved U$3 2.00 mm to (1.00, 110.0)
- moved U$4 2.00 mm to (1.00, 151.0)
- moved U$5 2.00 mm to (1.00, 192.0)
- moved U$6 2.00 mm to (1.00, 233.0)
- moved U$7 2.00 mm to (1.00, 69.0)
Connections:
- new net N$13: C3.1, U$10.2
- new net N$14: C3.2, U$10.3
- new net N$17: C7.1, U$12.2
- new net N$18: C7.2, U$12.3
- net GND: now also C4.2, C8.2, U$10.5, U$12.5; no longer U$9.3
- net SCL: now also U$10.8, U$12.8; no longer U$9.5
- net SDA: now also U$10.7, U$12.7; no longer U$9.6
- net VS: now also C4.1, C8.1, U$10.1, U$12.1; no longer U$9.4
Routing:
- net VS: track 31.1 -> 64.5 mm
- net SCL: track 40.7 -> 57.4 mm
- net SDA: track 42.6 -> 58.5 mm
- net N$10: track 76.7 -> 64.4 mm
- net POWER: track 136.9 -> 131.9 mm
- net N$18: track 0.00 -> 3.86 mm
- net N$14: track 0.00 -> 3.86 mm
- net N$13: track 0.00 -> 2.69 mm
- net N$17: track 0.00 -> 2.69 mm
- net GND: track 56.8 -> 56.9 mm, vias 4 -> 12
Other:
- outline, holes or cut-outs redrawn
