File: teams/power/Solar Panels/Side Panel V5/side panel V5.2.brd (EAGLE design)
At the start: 82 x 277.8 mm, 14 parts

Commit message: EPS/ old panels: Remove ground plane and changed temp sensor to TMP36
Parts:
- removed C3, C7: 100pF, Battery board V4.1 - simple signals:R0805
- removed C4, C8: (no value), Battery board V4.1 - simple signals:C0805
- removed U$10, U$12: TMP411, DubSat1 Components:TSSOP-8
- added C1, C2: (no value), DubSat1 Components:0805
- added CONN1, CONN3: PICOLOCK_6, DubSat1 Components:PICOLOCK_6
- U$2, U$8: value PICOLOCK_5 -> TMP36; device DubSat1 Components:PICOLOCK_5 -> DubSat1 Components:SOT-23-5
- moved U$8 14.3 mm to (17.0, 170.0), turned to 90 degrees
- moved U$2 13.0 mm to (65.0, 170.0)
Connections:
- removed net N$13: C3.1, U$10.2
- removed net N$14: C3.2, U$10.3
- removed net N$17: C7.1, U$12.2
- removed net N$18: C7.2, U$12.3
- removed net SCL: U$10.8, U$12.8, U$2.P$2, U$8.P$4
- removed net SDA: U$10.7, U$12.7, U$2.P$3, U$8.P$3
- removed net VS: C4.1, C8.1, U$10.1, U$12.1, U$2.P$1, U$8.P$5
- new net 3V3: C1.1, C2.1, CONN1.P$3, CONN3.P$3, U$2.P$2, U$2.P$4, U$8.P$2, U$8.P$4
- new net VOUT: CONN1.P$4, CONN3.P$1, CONN3.P$4, U$2.P$1, U$8.P$1
- net GND: now also C1.2, C2.2, CONN1.P$2, CONN1.P$5, CONN3.P$2, CONN3.P$5, U$8.P$5; no longer C4.2, C8.2, U$10.5, U$12.5, U$8.P$1
- net POWER: now also CONN1.P$1, CONN1.P$6, CONN3.P$6; no longer U$2.P$4, U$8.P$2
Routing:
- net VS: track 64.5 -> 0.00 mm
- net SDA: track 58.5 -> 0.00 mm
- net SCL: track 57.4 -> 0.00 mm
- net POWER: track 131.9 -> 108.8 mm
- net N$18: track 3.86 -> 0.00 mm
- net N$14: track 3.86 -> 0.00 mm
- net GND: track 56.9 -> 53.2 mm, vias 12 -> 4
- net N$13: track 2.69 -> 0.00 mm
- net N$17: track 2.69 -> 0.00 mm
- removed copper zone on layer 16, net GND
