File: teams/adcs/hardware/engineering_model/estimator/estimator_board.sch (EAGLE design)
At the start: 79 parts, among them U1 Value, U2 Value

Commit message: added two new capacitors to eagle library moved estimator, photodiode_center, and magetorquer board to their own foldr and created gerbers for them
Changed lines of the file:
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@@
 <pinref part="U1" gate="B" pin="AVSS2"/>
 <wire x1="83.82" y1="-45.72" x2="86.36" y2="-45.72" width="0.1524" layer="91"/>
+<junction x="86.36" y="-58.42"/>
+<junction x="86.36" y="-55.88"/>
+<junction x="86.36" y="-53.34"/>
+<junction x="86.36" y="-48.26"/>
+<junction x="86.36" y="-45.72"/>
 </segment>
 <segment>
@@
 <pinref part="U2" gate="B" pin="AVSS2"/>
 <wire x1="284.48" y1="-43.18" x2="287.02" y2="-43.18" width="0.1524" layer="91"/>
+<junction x="287.02" y="-43.18"/>
+<junction x="287.02" y="-45.72"/>
+<junction x="287.02" y="-50.8"/>
+<junction x="287.02" y="-53.34"/>
+<junction x="287.02" y="-55.88"/>
 </segment>
 <segment>
@@
 <wire x1="-99.06" y1="66.04" x2="-99.06" y2="68.58" width="0.1524" layer="91"/>
 <pinref part="SUPPLY6" gate="G$1" pin="3.3V"/>
+<junction x="-99.06" y="68.58"/>
 </segment>
 <segment>
@@
 <wire x1="96.52" y1="66.04" x2="96.52" y2="68.58" width="0.1524" layer="91"/>
 <pinref part="SUPPLY5" gate="G$1" pin="3.3V"/>
-</segment>
-<segment>
+<junction x="96.52" y="68.58"/>
+</segment>
+<segment>
