File: teams/adcs/hardware/engineering_model/flight_computer/flight_computer_board.sch (EAGLE design)
At the start: 85 parts, among them J1 FEMALE 2x3, U1 Value, U2 Value, U4 LINEAR_LDO_LT1761-X, U5 LINEAR_LDO_LT1761-X, U6 LINEAR_LDO_LT1761-X, U8 LINEAR_LDO_LT1761-X

Commit message: ADCS/FSW: Add LEDs to the BDOT MSP430
Parts:
- added D3, D4: (no value), DubSat1 Components:LED
- added R4, R8: (no value), DubSat1 Components:RESISTOR0805
- U$5: value BOARD_TEMPLATE -> BOARD_TEMPLATE1; device DubSat1 Components:BOARD_TEMPLATE -> DubSat1 Components:BOARD_TEMPLATE1
Connections:
- new net N$16: D4.C, R4.1
- new net N$18: D3.C, R8.1
- net BDOT_GND: now also R4.2, R8.2
- net N$5: now also D3.A
- net N$6: now also D4.A
Changed lines of the file:
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@@
 <layer number="59" name="tCarbon" color="7" fill="1" visible="no" active="no"/>
 <layer number="60" name="bCarbon" color="7" fill="1" visible="no" active="no"/>
+<layer number="88" name="SimResults" color="9" fill="1" visible="yes" active="yes"/>
+<layer number="89" name="SimProbes" color="9" fill="1" visible="yes" active="yes"/>
 <layer number="90" name="Modules" color="5" fill="1" visible="yes" active="yes"/>
 <layer number="91" name="Nets" color="2" fill="1" visible="yes" active="yes"/>
@@
 <part name="C16" library="rcl" library_urn="urn:adsk.eagle:library:334" deviceset="C-US" device="C0805" package3d_urn="urn:adsk.eagle:package:23617/2" value="4.7 nF"/>
 <part name="GND20" library="SparkFun-Aesthetics" deviceset="GND" device=""/>
-<part name="U$5" library="DubSat1 Components" deviceset="BOARD_TEMPLATE" device=""/>
+<part name="U$5" library="DubSat1 Components" deviceset="BOARD_TEMPLATE" device="1"/>
 <part name="U$6" library="DubSat1 Components" deviceset="PC104_CONNECTOR" device=""/>
 <part name="U$7" library="DubSat1 Components" deviceset="MSP-CAN_BLOCK" device=""/>
@@
 <part name="J1" library="SparkFun-Connectors" deviceset="CONN_03X2" device="FEMALE" value="FEMALE 2x3"/>
 <part name="J2" library="SparkFun-Connectors" deviceset="CONN_08X2" device=""/>
+<part name="D3" library="DubSat1 Components" deviceset="LED" device=""/>
+<part name="D4" library="DubSat1 Components" deviceset="LED" device=""/>
+<part name="R4" library="DubSat1 Components" deviceset="RESISTOR" device="0805"/>
+<part name="R8" library="DubSat1 Components" deviceset="RESISTOR" device="0805"/>
 </parts>
 <sheets>
@@
 <instance part="U$12" gate="G$1" x="-96.52" y="-15.24"/>
 <instance part="U$13" gate="G$1" x="-88.9" y="-198.12"/>
-<instance part="U$14" gate="G$1" x="208.28" y="154.94"/>
+<instance part="U$14" gate="G$1" x="254" y="154.94"/>
 <instance part="U$15" gate="G$1" x="358.14" y="170.18"/>
 <instance part="C18" gate="G$1" x="393.7" y="137.16" rot="R270"/>
@@
 <instance part="J1" gate="G$1" x="241.3" y="238.76"/>
 <instance part="J2" gate="G$1" x="213.36" y="-142.24"/>
+<instance part="D3" gate="G$1" x="215.9" y="172.72" rot="R180"/>
+<instance part="D4" gate="G$1" x="226.06" y="172.72" rot="R180"/>
+<instance part="R4" gate="G$1" x="226.06" y="185.42" rot="R90"/>
+<instance part="R8" gate="G$1" x="215.9" y="185.42" rot="R90"/>
 </instances>
 <busses>
@@
 <pinref part="U$7" gate="G$1" pin="P3.5_GPIO_DEBUG"/>
 <pinref part="U$14" gate="G$1" pin="P3.5_GPIO_DEBUG"/>
-<wire x1="170.18" y1="167.64" x2="190.5" y2="167.64" width="0.1524" layer="91"/>
+<wire x1="170.18" y1="167.64" x2="215.9" y2="167.64" width="0.1524" layer="91"/>
+<pinref part="D3" gate="G$1" pin="A"/>
+<wire x1="215.9" y1="167.64" x2="236.22" y2="167.64" width="0.1524" layer="91"/>
+<wire x1="215.9" y1="170.18" x2="215.9" y2="167.64" width="0.1524" layer="91"/>
+<junction x="215.9" y="167.64"/>
 </segment>
 </net>
@@
 <pinref part="U$7" gate="G$1" pin="P3.4_GPIO_DEBUG"/>
 <pinref part="U$14" gate="G$1" pin="P3.4_GPIO_DEBUG"/>
-<wire x1="170.18" y1="165.1" x2="190.5" y2="165.1" width="0.1524" layer="91"/>
+<wire x1="170.18" y1="165.1" x2="226.06" y2="165.1" width="0.1524" layer="91"/>
+<pinref part="D4" gate="G$1" pin="A"/>
+<wire x1="226.06" y1="165.1" x2="236.22" y2="165.1" width="0.1524" layer="91"/>
+<wire x1="226.06" y1="170.18" x2="226.06" y2="165.1" width="0.1524" layer="91"/>
+<junction x="226.06" y="165.1"/>
 </segment>
 </net>
@@
 <wire x1="185.42" y1="162.56" x2="185.42" y2="157.48" width="0.1524" layer="91"/>
 <pinref part="U$14" gate="G$1" pin="P2.1_RXD"/>
-<wire x1="185.42" y1="157.48" x2="190.5" y2="157.48" width="0.1524" layer="91"/>
+<wire x1="185.42" y1="157.48" x2="236.22" y2="157.48" width="0.1524" layer="91"/>
 </segment>
 </net>
@@
 <segment>
 <pinref part="U$14" gate="G$1" pin="P2.0_TXD"/>
-<wire x1="190.5" y1="154.94" x2="182.88" y2="154.94" width="0.1524" layer="91"/>
+<wire x1="236.22" y1="154.94" x2="182.88" y2="154.94" width="0.1524" layer="91"/>
 <wire x1="182.88" y1="154.94" x2="182.88" y2="160.02" width="0.1524" layer="91"/>
 <pinref part="U$7" gate="G$1" pin="P2.0_TXD"/>
@@
 <wire x1="180.34" y1="157.48" x2="180.34" y2="152.4" width="0.1524" layer="91"/>
 <pinref part="U$14" gate="G$1" pin="SBWTDIO"/>
-<wire x1="180.34" y1="152.4" x2="190.5" y2="152.4" width="0.1524" layer="91"/>
+<wire x1="180.34" y1="152.4" x2="236.22" y2="152.4" width="0.1524" layer="91"/>
 </segment>
 </net>
@@
 <segment>
 <pinref part="U$14" gate="G$1" pin="SBWTCK"/>
-<wire x1="190.5" y1="149.86" x2="177.8" y2="149.86" width="0.1524" layer="91"/>
+<wire x1="236.22" y1="149.86" x2="177.8" y2="149.86" width="0.1524" layer="91"/>
 <wire x1="177.8" y1="149.86" x2="177.8" y2="154.94" width="0.1524" layer="91"/>
 <wire x1="177.8" y1="154.94" x2="170.18" y2="154.94" width="0.1524" layer="91"/>
@@
 <segment>
 <pinref part="U$14" gate="G$1" pin="GND@1"/>
-<wire x1="190.5" y1="160.02" x2="187.96" y2="160.02" width="0.1524" layer="91"/>
-<wire x1="187.96" y1="160.02" x2="187.96" y2="144.78" width="0.1524" layer="91"/>
+<wire x1="236.22" y1="160.02" x2="233.68" y2="160.02" width="0.1524" layer="91"/>
+<wire x1="233.68" y1="160.02" x2="233.68" y2="144.78" width="0.1524" layer="91"/>
 <pinref part="U$14" gate="G$1" pin="GND@2"/>
-<wire x1="190.5" y1="162.56" x2="187.96" y2="162.56" width="0.1524" layer="91"/>
-<wire x1="187.96" y1="162.56" x2="187.96" y2="160.02" width="0.1524" layer="91"/>
-<junction x="187.96" y="160.02"/>
-<label x="187.96" y="144.78" size="1.778" layer="95" rot="R270" xref="yes"/>
+<wire x1="236.22" y1="162.56" x2="233.68" y2="162.56" width="0.1524" layer="91"/>
+<wire x1="233.68" y1="162.56" x2="233.68" y2="160.02" width="0.1524" layer="91"/>
+<junction x="233.68" y="160.02"/>
+<label x="233.68" y="144.78" size="1.778" layer="95" rot="R270" xref="yes"/>
 </segment>
 <segment>
@@
 <wire x1="33.02" y1="160.02" x2="38.1" y2="160.02" width="0.1524" layer="91"/>
 <label x="38.1" y="160.02" size="1.778" layer="95" xref="yes"/>
+</segment>
+<segment>
+<pinref part="R8" gate="G$1" pin="2"/>
+<wire x1="215.9" y1="190.5" x2="215.9" y2="193.04" width="0.1524" layer="91"/>
+<wire x1="215.9" y1="193.04" x2="226.06" y2="193.04" width="0.1524" layer="91"/>
+<pinref part="R4" gate="G$1" pin="2"/>
+<wire x1="226.06" y1="193.04" x2="236.22" y2="193.04" width="0.1524" layer="91"/>
+<wire x1="226.06" y1="190.5" x2="226.06" y2="193.04" width="0.1524" layer="91"/>
+<junction x="226.06" y="193.04"/>
+<label x="236.22" y="193.04" size="1.778" layer="95" xref="yes"/>
 </segment>
 </net>
@@
 </segment>
 </net>
+<net name="N$16" class="0">
+<segment>
+<pinref part="R4" gate="G$1" pin="1"/>
+<pinref part="D4" gate="G$1" pin="C"/>
+<wire x1="226.06" y1="177.8" x2="226.06" y2="180.34" width="0.1524" layer="91"/>
+</segment>
+</net>
+<net name="N$18" class="0">
+<segment>
+<pinref part="R8" gate="G$1" pin="1"/>
+<pinref part="D3" gate="G$1" pin="C"/>
+<wire x1="215.9" y1="177.8" x2="215.9" y2="180.34" width="0.1524" layer="91"/>
+</segment>
+</net>

Commit message: ADCS/MT: Update LDOs and stack board
Parts:
- U4, U5, U6, U8: value LINEAR_LDO_LT1761-X -> TPS732XX; device DubSat1 Components:LINEAR_LDO_LT1761-X -> DubSat1 Components:TPS732XX
Changed lines of the file:
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@@
 <part name="R7" library="DubSat1 Components" deviceset="RESISTOR" device="0805" value="10 kohm"/>
 <part name="R3" library="DubSat1 Components" deviceset="RESISTOR" device="0805" value="10 kohm"/>
-<part name="U4" library="DubSat1 Components" deviceset="LINEAR_LDO_LT1761-X" device=""/>
+<part name="U4" library="DubSat1 Components" deviceset="TPS732XX" device=""/>
 <part name="GND38" library="supply1" library_urn="urn:adsk.eagle:library:371" deviceset="GND" device=""/>
 <part name="C32" library="rcl" library_urn="urn:adsk.eagle:library:334" deviceset="C-US" device="C0805" package3d_urn="urn:adsk.eagle:package:23617/2" value="0.01 μF"/>
 <part name="C36" library="rcl" library_urn="urn:adsk.eagle:library:334" deviceset="C-US" device="C0805" package3d_urn="urn:adsk.eagle:package:23617/2" value="1 μF"/>
 <part name="C44" library="rcl" library_urn="urn:adsk.eagle:library:334" deviceset="C-US" device="C0805" package3d_urn="urn:adsk.eagle:package:23617/2" value="4.7 μF"/>
-<part name="U6" library="DubSat1 Components" deviceset="LINEAR_LDO_LT1761-X" device=""/>
+<part name="U6" library="DubSat1 Components" deviceset="TPS732XX" device=""/>
 <part name="GND44" library="supply1" library_urn="urn:adsk.eagle:library:371" deviceset="GND" device=""/>
 <part name="C48" library="rcl" library_urn="urn:adsk.eagle:library:334" deviceset="C-US" device="C0805" package3d_urn="urn:adsk.eagle:package:23617/2" value="0.01 μF"/>
 <part name="C49" library="rcl" library_urn="urn:adsk.eagle:library:334" deviceset="C-US" device="C0805" package3d_urn="urn:adsk.eagle:package:23617/2" value="1 μF"/>
 <part name="C51" library="rcl" library_urn="urn:adsk.eagle:library:334" deviceset="C-US" device="C0805" package3d_urn="urn:adsk.eagle:package:23617/2" value="4.7 μF"/>
-<part name="U5" library="DubSat1 Components" deviceset="LINEAR_LDO_LT1761-X" device=""/>
+<part name="U5" library="DubSat1 Components" deviceset="TPS732XX" device=""/>
 <part name="GND41" library="supply1" library_urn="urn:adsk.eagle:library:371" deviceset="GND" device=""/>
 <part name="C45" library="rcl" library_urn="urn:adsk.eagle:library:334" deviceset="C-US" device="C0805" package3d_urn="urn:adsk.eagle:package:23617/2" value="0.01 μF"/>
 <part name="C46" library="rcl" library_urn="urn:adsk.eagle:library:334" deviceset="C-US" device="C0805" package3d_urn="urn:adsk.eagle:package:23617/2" value="1 μF"/>
 <part name="C47" library="rcl" library_urn="urn:adsk.eagle:library:334" deviceset="C-US" device="C0805" package3d_urn="urn:adsk.eagle:package:23617/2" value="4.7 μF"/>
-<part name="U8" library="DubSat1 Components" deviceset="LINEAR_LDO_LT1761-X" device=""/>
+<part name="U8" library="DubSat1 Components" deviceset="TPS732XX" device=""/>
 <part name="GND50" library="supply1" library_urn="urn:adsk.eagle:library:371" deviceset="GND" device=""/>
 <part name="C55" library="rcl" library_urn="urn:adsk.eagle:library:334" deviceset="C-US" device="C0805" package3d_urn="urn:adsk.eagle:package:23617/2" value="0.01 μF"/>
