File: teams/adcs/hardware/engineering_model/flight_computer/flight_computer_board_CURRENT.sch (EAGLE design)
At the start: 89 parts, among them J1 FEMALE 2x3, U1 Value, U2 Value, U4 TPS732XX, U5 TPS732XX, U6 TPS732XX, U8 TPS732XX

Commit message: ADCS/FSW: Add on-board documentation
Connections:
- net N$12 renamed BDOT_RXD
- net N$13 renamed BDOT_TXD
- net N$14 renamed SBWTDIO
- net N$15 renamed SBWTCK
- net N$5 renamed BDOT_P3.5_GPIO_DEBUG
- net N$6 renamed BDOT_P3.4_GPIO_DEBUG
Changed lines of the file:
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@@
 <?xml version="1.0" encoding="utf-8"?>
 <!DOCTYPE eagle SYSTEM "eagle.dtd">
-<eagle version="8.4.3">
+<eagle version="8.6.0">
 <drawing>
 <settings>
@@
 </segment>
 </net>
-<net name="N$5" class="0">
+<net name="BDOT_P3.5_GPIO_DEBUG" class="0">
 <segment>
 <pinref part="U$7" gate="G$1" pin="P3.5_GPIO_DEBUG"/>
@@
 </segment>
 </net>
-<net name="N$6" class="0">
+<net name="BDOT_P3.4_GPIO_DEBUG" class="0">
 <segment>
 <pinref part="U$7" gate="G$1" pin="P3.4_GPIO_DEBUG"/>
@@
 </segment>
 </net>
-<net name="N$12" class="0">
+<net name="BDOT_RXD" class="0">
 <segment>
 <pinref part="U$7" gate="G$1" pin="P2.1_RXD"/>
@@
 </segment>
 </net>
-<net name="N$13" class="0">
+<net name="BDOT_TXD" class="0">
 <segment>
 <pinref part="U$14" gate="G$1" pin="P2.0_TXD"/>
@@
 </segment>
 </net>
-<net name="N$14" class="0">
+<net name="SBWTDIO" class="0">
 <segment>
 <pinref part="U$7" gate="G$1" pin="SBWTDIO"/>
@@
 </segment>
 </net>
-<net name="N$15" class="0">
+<net name="SBWTCK" class="0">
 <segment>
 <pinref part="U$14" gate="G$1" pin="SBWTCK"/>
