File: teams/power/Distribution Board/Distribution Board v3/distribution_board_v3.brd (EAGLE design)
At the start: 90 x 90 mm, 266 parts, among them U2 TPS732XX, U3 TPS732XX

Commit message: small changes to component values for distribution and generation board
Parts:
- C23, C32: value 0.01 μF -> .1u
- R102, R104, R105, R106, R107, R108, R11, R110, R111, R112, R114, R12, R13, R137, R138, R140, R142, R143, R144, R15, R16, R18, R22, R23, R24, R31, R32, R33, R46, R47, R48, R50, R52, R53, R64, R65, R66, R68, R69, R70, R77, R78, R80, R81, R82, R83, R97, R98: value (none) -> DNP
- R103, R109, R113, R139, R14, R141, R17, R29, R30, R49, R51, R67, R71, R79, R84, R99: value (none) -> 0
- R152, R6, R95: value 10 -> 500
- R5: value 10k -> 100
- R7: value 10 -> 5000

Commit message: updated i2c address on distribution board
Parts:
- R138: value DNP -> 0
- R139: value 0 -> DNP
- R28, R92: value DNP -> 100
Changed lines of the file:
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@@
 <layers>
 <layer number="1" name="Top" color="4" fill="1" visible="yes" active="yes"/>
-<layer number="2" name="Route2" color="11" fill="3" visible="no" active="yes"/>
-<layer number="3" name="Route3" color="4" fill="3" visible="no" active="yes"/>
+<layer number="2" name="Route2" color="11" fill="3" visible="yes" active="yes"/>
+<layer number="3" name="Route3" color="4" fill="3" visible="yes" active="yes"/>
 <layer number="4" name="Route4" color="1" fill="4" visible="no" active="no"/>
 <layer number="5" name="Route5" color="4" fill="4" visible="no" active="no"/>
@@
 <layer number="29" name="tStop" color="7" fill="3" visible="no" active="yes"/>
 <layer number="30" name="bStop" color="7" fill="6" visible="no" active="yes"/>
-<layer number="31" name="tCream" color="7" fill="4" visible="yes" active="yes"/>
+<layer number="31" name="tCream" color="7" fill="4" visible="no" active="yes"/>
 <layer number="32" name="bCream" color="7" fill="5" visible="no" active="yes"/>
 <layer number="33" name="tFinish" color="6" fill="3" visible="no" active="yes"/>
@@
 <element name="U$8" library="DubSat1 Components" package="SOT-323" value="DMN5L06WK" x="-34" y="8"/>
 <element name="U$9" library="DubSat1 Components" package="POWERDI5060-8" value="DMP2002UPS" x="-41" y="8"/>
-<element name="R28" library="DubSat1 Components" package="0805" value="DNP" x="-37" y="2" rot="R270"/>
+<element name="R28" library="DubSat1 Components" package="0805" value="100" x="-37" y="2" rot="R270"/>
 <element name="C9" library="DubSat1 Components" package="0805" value="DNP" x="-34" y="3"/>
 <element name="C10" library="DubSat1 Components" package="0805" value="DNP" x="-34" y="1"/>
@@
 <attribute name="NAME" x="-13.238675" y="7.79969375" size="0.4064" layer="25" font="vector" rot="R270"/>
 </element>
-<element name="R138" library="DubSat1 Components" package="0805" value="DNP" x="-18.133" y="4.668" smashed="yes" rot="R270">
+<element name="R138" library="DubSat1 Components" package="0805" value="0" x="-18.133" y="4.668" smashed="yes" rot="R270">
 <attribute name="NAME" x="-18.318675" y="4.87069375" size="0.4064" layer="25" font="vector" rot="R270"/>
 </element>
-<element name="R139" library="DubSat1 Components" package="0805" value="0" x="-12.418" y="4.668" smashed="yes" rot="R270">
+<element name="R139" library="DubSat1 Components" package="0805" value="DNP" x="-12.418" y="4.668" smashed="yes" rot="R270">
 <attribute name="NAME" x="-12.603675" y="4.87069375" size="0.4064" layer="25" font="vector" rot="R270"/>
 </element>
@@
 <element name="U$17" library="DubSat1 Components" package="SOT-323" value="DMN5L06WK" x="30.5" y="15"/>
 <element name="U$18" library="DubSat1 Components" package="POWERDI5060-8" value="DMP2002UPS" x="23.5" y="15"/>
-<element name="R92" library="DubSat1 Components" package="0805" value="DNP" x="27.5" y="9" rot="R270"/>
+<element name="R92" library="DubSat1 Components" package="0805" value="100" x="27.5" y="9" rot="R270"/>
 <element name="C48" library="DubSat1 Components" package="0805" value="DNP" x="30.5" y="10"/>
 <element name="C49" library="DubSat1 Components" package="0805" value="DNP" x="30.5" y="8"/>
