File: teams/power/Gen Board/Generation Board v5/generation_board_v5.brd (EAGLE design)
At the start: 90 x 90 mm, 218 parts, among them U2 LT3652, U3 LT3652, U4 LT3652, U5 TPS732XX, U7 TPS732XX

Commit message: small changes to component values for distribution and generation board
Parts:
- R101, R102, R104, R105, R106, R107, R15, R16, R29, R32, R33, R34, R73, R74, R75, R77, R79, R80: value (none) -> DNP
- R103, R108, R112, R2, R30, R31, R76, R78, R84: value (none) -> 0
- R111, R37, R83: value (none) -> .1
- R17, R61, R89: value 520k -> 523k
- R19, R91: value .067 -> .09
- R20, R64, R92: value 545k -> 604k
- R21, R93: value 545k -> 143k
- R63: value .067 -> .11
- R65: value 545k -> 182k

Commit message: fixed component values
Parts:
- R25, R26, R69, R70, R97, R98: value 5k -> 1.3k
- R60, R8, R88: value DNP -> 0
Changed lines of the file:
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@@
 <layer number="28" name="bValues" color="7" fill="1" visible="yes" active="yes"/>
 <layer number="29" name="tStop" color="7" fill="3" visible="no" active="yes"/>
-<layer number="30" name="bStop" color="7" fill="6" visible="yes" active="yes"/>
+<layer number="30" name="bStop" color="7" fill="6" visible="no" active="yes"/>
 <layer number="31" name="tCream" color="7" fill="4" visible="yes" active="yes"/>
 <layer number="32" name="bCream" color="7" fill="5" visible="no" active="yes"/>
@@
 <element name="U$5" library="DubSat1 Components" package="SOT-323" value="DMN5L06WK" x="-19.75" y="-37"/>
 <element name="U$9" library="DubSat1 Components" package="POWERDI5060-8" value="DMP2002UPS" x="-26.75" y="-37"/>
-<element name="R8" library="DubSat1 Components" package="0805" value="DNP" x="-15.75" y="-36" rot="R180"/>
+<element name="R8" library="DubSat1 Components" package="0805" value="0" x="-15.75" y="-36" rot="R180"/>
 <element name="C5" library="DubSat1 Components" package="0805" value="DNP" x="-14.75" y="-39" rot="R270"/>
 <element name="C6" library="DubSat1 Components" package="0805" value="DNP" x="-16.75" y="-39" rot="R270"/>
@@
 <attribute name="NAME" x="-19.75069375" y="-13.315675" size="0.4064" layer="25" font="vector"/>
 </element>
-<element name="R26" library="DubSat1 Components" package="0805" value="5k" x="-18.04" y="-16.31" smashed="yes" rot="R180">
+<element name="R26" library="DubSat1 Components" package="0805" value="1.3k" x="-18.04" y="-16.31" smashed="yes" rot="R180">
 <attribute name="NAME" x="-18.225675" y="-15.72630625" size="0.4064" layer="25" font="vector" rot="R270"/>
 </element>
@@
 <attribute name="NAME" x="-22.54369375" y="-22.535675" size="0.4064" layer="25" font="vector"/>
 </element>
-<element name="R25" library="DubSat1 Components" package="0805" value="5k" x="-17.99" y="-18.53" smashed="yes" rot="R180">
+<element name="R25" library="DubSat1 Components" package="0805" value="1.3k" x="-17.99" y="-18.53" smashed="yes" rot="R180">
 <attribute name="NAME" x="-18.175675" y="-17.94630625" size="0.4064" layer="25" font="vector" rot="R270"/>
 </element>
@@
 <element name="U$15" library="DubSat1 Components" package="SOT-323" value="DMN5L06WK" x="4.25" y="-37"/>
 <element name="U$16" library="DubSat1 Components" package="POWERDI5060-8" value="DMP2002UPS" x="-2.75" y="-37"/>
-<element name="R60" library="DubSat1 Components" package="0805" value="DNP" x="8.25" y="-36" rot="R180"/>
+<element name="R60" library="DubSat1 Components" package="0805" value="0" x="8.25" y="-36" rot="R180"/>
 <element name="C40" library="DubSat1 Components" package="0805" value="DNP" x="9.25" y="-39" rot="R270"/>
 <element name="C41" library="DubSat1 Components" package="0805" value="DNP" x="7.25" y="-39" rot="R270"/>
@@
 <attribute name="NAME" x="4.24930625" y="-13.315675" size="0.4064" layer="25" font="vector"/>
 </element>
-<element name="R70" library="DubSat1 Components" package="0805" value="5k" x="5.96" y="-16.31" smashed="yes" rot="R180">
+<element name="R70" library="DubSat1 Components" package="0805" value="1.3k" x="5.96" y="-16.31" smashed="yes" rot="R180">
 <attribute name="NAME" x="5.774325" y="-15.72630625" size="0.4064" layer="25" font="vector" rot="R270"/>
 </element>
@@
 <attribute name="NAME" x="1.45630625" y="-22.535675" size="0.4064" layer="25" font="vector"/>
 </element>
-<element name="R69" library="DubSat1 Components" package="0805" value="5k" x="6.01" y="-18.53" smashed="yes" rot="R180">
+<element name="R69" library="DubSat1 Components" package="0805" value="1.3k" x="6.01" y="-18.53" smashed="yes" rot="R180">
 <attribute name="NAME" x="5.824325" y="-17.94630625" size="0.4064" layer="25" font="vector" rot="R270"/>
 </element>
@@
 <element name="U$21" library="DubSat1 Components" package="SOT-323" value="DMN5L06WK" x="25" y="-37.25"/>
 <element name="U$22" library="DubSat1 Components" package="POWERDI5060-8" value="DMP2002UPS" x="18" y="-37.25"/>
-<element name="R88" library="DubSat1 Components" package="0805" value="DNP" x="29" y="-36.25" rot="R180"/>
+<element name="R88" library="DubSat1 Components" package="0805" value="0" x="29" y="-36.25" rot="R180"/>
 <element name="C59" library="DubSat1 Components" package="0805" value="DNP" x="30" y="-39.25" rot="R270"/>
 <element name="C60" library="DubSat1 Components" package="0805" value="DNP" x="28" y="-39.25" rot="R270"/>
@@
 <attribute name="NAME" x="28.24930625" y="-13.315675" size="0.4064" layer="25" font="vector"/>
 </element>
-<element name="R98" library="DubSat1 Components" package="0805" value="5k" x="29.96" y="-16.31" smashed="yes" rot="R180">
+<element name="R98" library="DubSat1 Components" package="0805" value="1.3k" x="29.96" y="-16.31" smashed="yes" rot="R180">
 <attribute name="NAME" x="29.774325" y="-15.72630625" size="0.4064" layer="25" font="vector" rot="R270"/>
 </element>
@@
 <attribute name="NAME" x="25.45630625" y="-22.535675" size="0.4064" layer="25" font="vector"/>
 </element>
-<element name="R97" library="DubSat1 Components" package="0805" value="5k" x="30.01" y="-18.53" smashed="yes" rot="R180">
+<element name="R97" library="DubSat1 Components" package="0805" value="1.3k" x="30.01" y="-18.53" smashed="yes" rot="R180">
 <attribute name="NAME" x="29.824325" y="-17.94630625" size="0.4064" layer="25" font="vector" rot="R270"/>
 </element>

Commit message: minor changes
Connections:
- net ENABLE_PT1 renamed DISABLE_PT1
- new net DISABLE_PT2: BLK1.P3.6_GPIO/PWM
- new net DISABLE_PT3: BLK1.P2.6_GPIO/PWM
- net ENABLE_PT2: no longer BLK1.P3.6_GPIO/PWM
- net ENABLE_PT3: no longer BLK1.P2.6_GPIO/PWM
Routing:
- net ENABLE_PT2: track 69.9 -> 63.1 mm
Changed lines of the file:
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@@
 <wire x1="-22.80375" y1="-19.5748" x2="-22.6252" y2="-19.39625" width="0.2032" layer="1"/>
 </signal>
-<signal name="ENABLE_PT1">
+<signal name="DISABLE_PT1">
 <contactref element="R23" pad="2"/>
 <contactref element="LT3652_DISABLE1" pad="1"/>
@@
 <wire x1="1.973" y1="-23.317" x2="2.04" y2="-23.25" width="0.1524" layer="1"/>
 <wire x1="1.973" y1="-23.317" x2="-0.104" y2="-23.017" width="0.1524" layer="1"/>
-<contactref element="BLK1" pad="P3.6_GPIO/PWM"/>
 <wire x1="2.04" y1="-23.25" x2="3.6902" y2="-21.5998" width="0.2032" layer="1"/>
 <wire x1="3.6902" y1="-21.5998" x2="3.6902" y2="-20.85875" width="0.2032" layer="1"/>
@@
 <via x="30" y="16" extent="1-16" drill="0.35"/>
 <wire x1="30" y1="16" x2="30.75" y2="16.75" width="0.2032" layer="1"/>
-<wire x1="30.75" y1="16.75" x2="30.75" y2="23.6" width="0.2032" layer="1"/>
 </signal>
 <signal name="N$23">
@@
 <wire x1="25.973" y1="-23.317" x2="26.04" y2="-23.25" width="0.1524" layer="1"/>
 <wire x1="25.973" y1="-23.317" x2="23.896" y2="-23.017" width="0.1524" layer="1"/>
-<contactref element="BLK1" pad="P2.6_GPIO/PWM"/>
 <wire x1="26.04" y1="-23.25" x2="27.6902" y2="-21.5998" width="0.2032" layer="1"/>
 <wire x1="27.6902" y1="-21.5998" x2="27.6902" y2="-20.85875" width="0.2032" layer="1"/>
@@
 <wire x1="38" y1="2.5" x2="38" y2="6.8340875" width="0.2032" layer="1"/>
 <wire x1="35.50125" y1="20.2398" x2="34.6702" y2="20.2398" width="0.2032" layer="1"/>
-<wire x1="34.6702" y1="20.2398" x2="34.6" y2="20.25" width="0.2032" layer="1"/>
 <wire x1="38" y1="6.8340875" x2="38.4064" y2="7.2404875" width="0.2032" layer="1"/>
 <wire x1="38.4064" y1="7.2404875" x2="38.4064" y2="17.27465" width="0.2032" layer="1"/>
@@
 <via x="10.47" y="28.03" extent="1-16" drill="0.35"/>
 </signal>
+<signal name="DISABLE_PT2">
+<contactref element="BLK1" pad="P3.6_GPIO/PWM"/>
+</signal>
+<signal name="DISABLE_PT3">
+<contactref element="BLK1" pad="P2.6_GPIO/PWM"/>
+</signal>
 </signals>
