File: teams/adcs/hardware/flight_model/flight_computer/flight_computer_board_f1.sch (EAGLE design)
At the start: 89 parts, among them J1 FEMALE 2x3, U1 Value, U2 Value, U4 TPS732XX, U5 TPS732XX, U6 TPS732XX, U8 TPS732XX

Commit message: ADCS/FSW: Add debug header and LEDs to 430
Parts:
- removed C1: 0.1uF, rcl:C-USC0805
- removed C10, C11, C12, C40, C41, C42, C43, C9: 13 pF, rcl:C-USC0805
- removed C22: 0.22 uF, rcl:C-USC0805
- removed C23, C24, C25, C27, C28, C3, C33, C35, C37, C39, C5, C50, C6, C8: 0.1 uF, rcl:C-USC0805
- removed C26, C34, C38, C4, C7: 4.7 uF, rcl:C-USC0805
- removed J2: (no value), SparkFun-Connectors:CONN_08X2
- removed R10, R9: 10 kohm, DubSat1 Components:RESISTOR0805
- removed SDO/SA1: 0_OHM_JUMPER, DubSat1 Components:0_OHM_JUMPER
- removed U$10, U$8: CAN_BLOCK, DubSat1 Components:CAN_BLOCK
- removed U$11, U$12, U$13, U$3: M20, SparkFun-Connectors:M20
- removed U$17: LSM6DSM, LSM6DSM:LSM6DSM
- removed U$18: HMC5983, DubSat1 Components:HMC5983
- removed U$2, U$9: EPSON_CRYSTAL_FA-238, DubSat1 Components:EPSON_CRYSTAL_FA-238
- removed U$4: EPSON_CRYSTAL_FC-135R, DubSat1 Components:EPSON_CRYSTAL_FC-135R
- removed U1, U2: Value, DubSat1 Components:MSP432P401R_PZ
- added BLK1: MSP-CAN_BLOCK, DubSat1 Components:MSP-CAN_BLOCK
- R1, R2: value 330 ohm -> (none)
- U$1: value EPSON_CRYSTAL_FC-135R -> PROGRAM/DEBUG_PORT; device DubSat1 Components:EPSON_CRYSTAL_FC-135R -> DubSat1 Components:PROGRAM/DEBUG_PORT
Connections:
- removed net BCLUART_RXD1: U$12.8, U$3.8, U1A.P1.2_UCA0RXD_UCA0SOMI
- removed net BCLUART_RXD2: U$11.8, U$13.8, U2A.P1.2_UCA0RXD_UCA0SOMI
- removed net BCLUART_TXD1: U$12.7, U$3.7, U1A.P1.3_UCA0TXD_UCA0SIMO
- removed net BCLUART_TXD2: U$11.7, U$13.7, U2A.P1.3_UCA0TXD_UCA0SIMO
- removed net CAN-INT1: U$12.15, U$3.15, U$8.INT, U1A.P1.0_UCA0STE
- removed net CAN-INT2: U$10.INT, U$11.15, U$13.15
- removed net CANINT2: U2A.P1.0_UCA0STE
- removed net ESTIMAT_DRDY: J2.14, U$18.DRDY
- removed net ESTIMAT_DRDY_JP: J2.13, U2A.P4.5_A8
- removed net ESTIMAT_IMU_INT1_JP: U2A.P4.6_A7
- removed net ESTIMAT_INU_INT2_JP: U2A.P4.7_A6
- removed net ESTIMAT_SCL_IMU: J2.6, U$11.5, U$13.5, U$17.SCL
- removed net ESTIMAT_SCL_JP: J2.1, J2.5, R10.2, U2A.P6.5_UCB1SOMI_UCB1SCL_C1.2
- removed net ESTIMAT_SCL_MAG: J2.2, U$18.SCL/SPI_SCK
- removed net ESTIMAT_SDA_IMU: J2.8, U$17.SDA
- removed net ESTIMAT_SDA_JP: J2.3, J2.7, R9.2, U2A.P6.4_UCB1SIMO_UCB1SDA_C1.3
- removed net ESTIMAT_SDA_MAG: J2.4, U$11.4, U$13.4, U$18.SDA/SPI_SDI
- removed net ESTIMAT_SOC: J2.16, U$18.SOC
- removed net ESTIMAT_SOC_JP: J2.15, U2A.P4.1_A12
- removed net I2C_SCL1: U$12.5, U$3.5, U1A.P6.5_UCB1SOMI_UCB1SCL_C1.2
- removed net I2C_SDA1: U$12.4, U$3.4, U1A.P6.4_UCB1SIMO_UCB1SDA_C1.3
- removed net IMU_INT1: J2.10, U$17.INT1
- removed net IMU_INT1_JP: J2.9
- removed net IMU_INT2: J2.12, U$17.INT2
- removed net IMU_INT2_JP: J2.11
- removed net N$10: C12.1, U$2.P$3, U1A.PJ.2_HFXOUT
- removed net N$11: C11.1, U$2.P$1, U1A.PJ.3_HFXIN
- removed net N$25: SDO/SA1.SIG, U$17.SDO/SA0
- removed net N$3: D1.A, U1A.P2.0_PM_UCA1STE
- removed net N$34: C26.1, U$18.C1
- removed net N$35: C22.2, U$18.SETP
- removed net N$36: C22.1, U$18.SETC
- removed net N$4: D1.C, R1.1
- removed net N$40: C40.1, U$4.P$1, U2A.PJ.1_LFXOUT
- removed net N$41: C41.1, U$4.P$2, U2A.PJ.0_LFXIN
- removed net N$42: C42.1, U$9.P$1, U2A.PJ.3_HFXIN
- removed net N$43: C43.1, U$9.P$3, U2A.PJ.2_HFXOUT
- removed net N$7: C3.1, U1B.VCORE
- removed net N$8: C10.1, U$1.P$2, U1A.PJ.0_LFXIN
- removed net N$9: C9.1, U$1.P$1, U1A.PJ.1_LFXOUT
- removed net RST1: U$12.9, U$3.9, U1A.RST_NMI_N
- removed net RST2: U$11.9, U$13.9, U2A.RST_NMI_N
- removed net SPI-CLK1: U$12.17, U$3.17, U$8.SCLK, U1A.P1.5_UCB0CLK
- removed net SPI-CLK2: U$10.SCLK, U$11.17, U$13.17, U2A.P1.5_UCB0CLK
- removed net SPI-CS1: U$12.16, U$3.16, U$8.CS, U1A.P1.4_UCB0STE
- removed net SPI-CS2: U$10.CS, U$11.16, U$13.16, U2A.P1.4_UCB0STE
- removed net SPI-MISO1: U$12.19, U$3.19, U$8.MISO, U1A.P1.7_UCB0SOMI_UCB0SCL
- removed net SPI-MISO2: U$10.MISO, U$11.19, U$13.19, U2A.P1.7_UCB0SOMI_UCB0SCL
- removed net SPI-MOSI1: U$12.18, U$3.18, U$8.MOSI, U1A.P1.6_UCB0SIMO_UCB0SDA
- removed net SPI-MOSI2: U$10.MOSI, U$11.18, U$13.18, U2A.P1.6_UCB0SIMO_UCB0SDA
- removed net TCK_SWDCLK1: U$12.10, U$3.10, U1A.SWCLKTCK
- removed net TCK_SWDCLK2: U$11.10, U$13.10, U2A.SWCLKTCK
- removed net TDI1: U$12.13, U$3.13, U1A.PJ.4_TDI_ADC14CLK
- removed net TDI2: U$11.13, U$13.13, U2A.PJ.4_TDI_ADC14CLK
- removed net TDO1: U$12.12, U$3.12, U1A.PJ.5_TDO_SWO
- removed net TDO2: U$11.12, U$13.12, U2A.PJ.5_TDO_SWO
- removed net TMS_SWDIO1: U$12.11, U$3.11, U1A.SWDIOTMS
- removed net TMS_SWDIO2: U$11.11, U$13.11, U2A.SWDIOTMS
- removed net UART_RXD1: U$12.2, U$3.2, U1A.P3.2_PM_UCA2RXD_PM_UCA2SOMI
- removed net UART_RXD2: U$11.2, U$13.2, U2A.P3.2_PM_UCA2RXD_PM_UCA2SOMI
- removed net UART_TXD1: U$12.1, U$3.1, U1A.P3.3_PM_UCA2TXD_PM_UCA2SIMO
- removed net UART_TXD2: U$11.1, U$13.1, U2A.P3.3_PM_UCA2TXD_PM_UCA2SIMO
- removed net VCORE: C33.1, U2B.VCORE
- new net BDOT_SBWTCK: U$14.SBWTCK, U$7.SBWTCK
- new net BDOT_SBWTDIO: U$14.SBWTDIO, U$7.SBWTDIO
- new net ESTIMAT_BRIDGE_I2C_SCL_2: BLK1.P7.1_I2C-SCL-2
- new net ESTIMAT_BRIDGE_I2C_SDA_2: BLK1.P7.0_I2C-SDA-2
- new net P3.4_GPIO_DEBUG: BLK1.P3.4_GPIO_DEBUG, D1.A, U$1.P3.4_GPIO_DEBUG
- new net P3.5_GPIO_DEBUG: BLK1.P3.5_GPIO_DEBUG, D2.A, U$1.P3.5_GPIO_DEBUG
- new net RXD: BLK1.P2.1_RXD, U$1.P2.1_RXD
- new net TXD: BLK1.P2.0_TXD, U$1.P2.0_TXD
- net CANH: now also BLK1.CANH; no longer U$10.CANH, U$8.CANH
- net CANL: now also BLK1.CANL; no longer U$10.CANL, U$8.CANL
- net ESTIMAT_3V3: now also BLK1.3.3V_CAN@1, BLK1.3.3V_CAN@2, BLK1.3.3V_MSP-ANALOG@1, BLK1.3.3V_MSP@2, BLK1.3.3V_MSP@3; no longer C1.1, C23.1, C24.1, C25.2, C27.1, C28.1, C34.1, C35.1, C37.1, C38.1, C39.1, C4.1, C5.1, C50.1, C6.1, C7.1, C8.1, R10.1, R9.1, SDO/SA1.VCC, U$10.3.3V@1, U$10.3.3V@2, U$17.CS, U$17.VDD, U$17.VDDIO, U$18.!SPI_CS, U$18.I2C/!SPI, U$18.VDD, U$18.VDDIO, U$8.3.3V@1, U$8.3.3V@2, U1B.AVCC1, U1B.AVCC2, U1B.DVCC1, U1B.DVCC2, U2B.AVCC1, U2B.AVCC2, U2B.DVCC1, U2B.DVCC2
- net ESTIMAT_5V: now also BLK1.5V_CAN; no longer U$10.5V, U$8.5V
- net ESTIMAT_GND: now also BLK1.GND, U$1.GND@1, U$1.GND@2; no longer C1.2, C10.2, C11.2, C12.2, C23.2, C24.2, C25.1, C26.2, C27.2, C28.2, C3.2, C33.2, C34.2, C35.2, C37.2, C38.2, C39.2, C4.2, C40.2, C41.2, C42.2, C43.2, C5.2, C50.2, C6.2, C7.2, C8.2, C9.2, SDO/SA1.GND, U$10.GND, U$11.14, U$11.20, U$11.3, U$11.6, U$12.14, U$12.20, U$12.3, U$12.6, U$13.14, U$13.20, U$13.3, U$13.6, U$17.GND@1, U$17.GND@2, U$17.SCX, U$17.SDX, U$18.GND, U$3.14, U$3.20, U$3.3, U$3.6, U$8.GND, U1B.AVSS1, U1B.AVSS2, U1B.AVSS3, U1B.DVSS1, U1B.DVSS2, U1B.DVSS3, U2B.AVSS1, U2B.AVSS2, U2B.AVSS3, U2B.DVSS1, U2B.DVSS2, U2B.DVSS3
- net N$1: now also D2.C, R1.1; no longer D2.A, U2A.P2.0_PM_UCA1STE
- net N$2: now also D1.C; no longer D2.C
- net SBWTCK: now also BLK1.SBWTCK, U$1.SBWTCK; no longer U$14.SBWTCK, U$7.SBWTCK
- net SBWTDIO: now also BLK1.SBWTDIO, U$1.SBWTDIO; no longer U$14.SBWTDIO, U$7.SBWTDIO
- net SYNC1: no longer U1A.P5.0_A5, U2A.P5.0_A5
- net SYNC2: no longer U1A.P5.1_A4, U2A.P5.1_A4
Other:
- note removed: "Estimator IMU"
- note removed: "Estimator Magnetometer"
- note removed: "Estimator sensor config jumper"
- note removed: "MCU specific Debug/Programming"
- note removed: "Power/Smoothing for U1"
- note removed: "Power/Smoothing for U2"
- moved on the sheet: D1, D2, R1, R2

Commit message: ADCS/FSW: Remove SYNC connections to BDOT
Parts:
- added BLK2: MSP-CAN_BLOCK, DubSat1 Components:MSP-CAN_BLOCK
- added D5, D6: (no value), DubSat1 Components:LED
- added R10, R9: (no value), DubSat1 Components:RESISTOR0805
- added U$2: PROGRAM/DEBUG_PORT, DubSat1 Components:PROGRAM/DEBUG_PORT
Connections:
- removed net ESTIMAT_BRIDGE_I2C_SCL_2: BLK1.P7.1_I2C-SCL-2
- removed net ESTIMAT_BRIDGE_I2C_SDA_2: BLK1.P7.0_I2C-SDA-2
- new net N$3: D6.C, R9.1
- new net N$4: D5.C, R10.1
- new net P3.4_GPIO_DEBUG1: BLK2.P3.4_GPIO_DEBUG, D5.A, U$2.P3.4_GPIO_DEBUG
- new net P3.5_GPIO_DEBUG1: BLK2.P3.5_GPIO_DEBUG, D6.A, U$2.P3.5_GPIO_DEBUG
- new net RXD1: BLK2.P2.1_RXD, U$2.P2.1_RXD
- new net SBWTCK1: BLK2.SBWTCK, U$2.SBWTCK
- new net SBWTDIO1: BLK2.SBWTDIO, U$2.SBWTDIO
- new net TXD1: BLK2.P2.0_TXD, U$2.P2.0_TXD
- net CANH: now also BLK2.CANH
- net CANL: now also BLK2.CANL
- net ESTIMAT_3V3: now also BLK2.3.3V_CAN@1, BLK2.3.3V_CAN@2, BLK2.3.3V_MSP-ANALOG@1, BLK2.3.3V_MSP@2, BLK2.3.3V_MSP@3
- net ESTIMAT_5V: now also BLK2.5V_CAN
- net ESTIMAT_GND: now also BLK2.GND, R10.2, R9.2, U$2.GND@1, U$2.GND@2
- net SYNC1: no longer U$7.P7.2_SYNC1
- net SYNC2: no longer U$7.PJ.3_SYNC2
