File: teams/propulsion/flight/controller/PPT_controller_flight1.sch (EAGLE design)
At the start: 32 parts, among them U2 TPS732XX, U4 TPS732XX

Commit message: PPT Controller Board Revisions
Revisions to the PPT Controller Board to reflect the mirroring of the PC-104. CAN routing has been addressed and a diode added to the Charge Board trace. DubSat-1 Components library change is to add Paige's diode to the library.
Parts:
- added 0.1U: 0.1u, DubSat1 Components:CAPACITOR0805
- added 1U: 1u, DubSat1 Components:CAPACITOR0805
- added D4: LLP1006-2L, DubSat1 Components:LLP1006-2L
Connections:
- net 3.3V: now also 0.1U.2, 1U.2, BLK1.3.3V_MSP-ANALOG@1
- net CHARGE_BOARD_VBAT: now also D4.P$2
- net GND: now also D4.P$1
