File: teams/power/Flight/Generation/generation_board_f1.brd (EAGLE design)
At the start: 90 x 90 mm, 229 parts, among them U2 LT3652, U3 LT3652, U4 LT3652, U5 TPS732XX, U7 TPS732XX

Commit message: Flight merge (#230)
Merge of the flight code into master
Routing:
- net 3.3V: track 360.5 -> 378.1 mm, vias 12 -> 18
- net DEPLOY_EN: vias 2 -> 6
Changed lines of the file:
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@@
 <wire x1="-1" y1="36.5" x2="-0.54" y2="36.96" width="0.2032" layer="3"/>
 <wire x1="-0.54" y1="36.96" x2="1.27" y2="36.96" width="0.2032" layer="3"/>
-<wire x1="-1" y1="36.5" x2="-1.27" y2="36.96" width="0" layer="19" extent="1-3"/>
-<wire x1="7.25" y1="-38.1" x2="5.9159125" y2="-37.7" width="0" layer="19" extent="1-3"/>
+<via x="7.25" y="-37.5" extent="1-16" drill="0.35"/>
+<via x="28.1" y="-37.7" extent="1-16" drill="0.35"/>
+<via x="7.77" y="-37.47" extent="1-16" drill="0.35"/>
+<via x="-17.14" y="-36.697" extent="1-16" drill="0.35"/>
+<wire x1="-17.5" y1="-36.317" x2="-17.14" y2="-36.697" width="0" layer="19" extent="1-3"/>
+<wire x1="28.1" y1="-37.7" x2="28.1" y2="-38.1" width="0" layer="19" extent="1-1"/>
+<wire x1="-1.27" y1="36.96" x2="-1" y2="36.5" width="0" layer="19" extent="1-3"/>
+<wire x1="7.25" y1="-37.5" x2="5.9159125" y2="-37.7" width="0" layer="19" extent="1-3"/>
+<wire x1="7.35" y1="-38" x2="7.25" y2="-37.5" width="0" layer="19" extent="1-1"/>
+<wire x1="7.77" y1="-37.47" x2="7.25" y2="-37.5" width="0" layer="19" extent="1-1"/>
 </signal>
 <signal name="N$2">
@@
 <wire x1="35.5" y1="-10.5" x2="36" y2="-10" width="0.2032" layer="3"/>
 <wire x1="36" y1="-10" x2="40" y2="-10" width="0.2032" layer="3"/>
-<wire x1="40" y1="-10" x2="40" y2="-33" width="0.2032" layer="3"/>
 <wire x1="-39" y1="-33" x2="-40" y2="-32" width="0.2032" layer="3"/>
 <wire x1="-40" y1="-11" x2="-40" y2="10" width="0.2032" layer="3"/>
@@
 <wire x1="-40" y1="-11" x2="-40" y2="-32" width="0.2032" layer="3"/>
 <wire x1="-40" y1="10" x2="-40" y2="29" width="0.2032" layer="3"/>
-<wire x1="-40" y1="29" x2="-40" y2="30.9025" width="0.2032" layer="1"/>
+<wire x1="-40" y1="29" x2="-40" y2="30.9025" width="0.3048" layer="1"/>
 <wire x1="12.25" y1="-33" x2="-12" y2="-33" width="0.2032" layer="3"/>
 <wire x1="12.25" y1="-33" x2="36.25" y2="-33" width="0.2032" layer="3"/>
-<wire x1="36.25" y1="-33" x2="40" y2="-33" width="0.2032" layer="3"/>
 <wire x1="-12" y1="-33" x2="-39" y2="-33" width="0.2032" layer="3"/>
 <wire x1="-36.5" y1="10" x2="-35.5" y2="10" width="0.2032" layer="1"/>
@@
 <contactref element="R42" pad="2"/>
 <contactref element="R43" pad="2"/>
-<wire x1="-2.1" y1="22.5" x2="-2.1" y2="20.25" width="0.2032" layer="1"/>
-<wire x1="-2.1" y1="20.25" x2="3" y2="15.75" width="0.2032" layer="1"/>
-<wire x1="3" y1="15.75" x2="4" y2="14.75" width="0.2032" layer="1"/>
+<wire x1="-2.1" y1="22.5" x2="-2.1" y2="20.25" width="0.3048" layer="1"/>
+<wire x1="-2.1" y1="20.25" x2="3" y2="15.75" width="0.3048" layer="1"/>
+<wire x1="3" y1="15.75" x2="4" y2="14.75" width="0.3048" layer="1"/>
+<wire x1="-40" y1="29" x2="-38.75" y2="27.75" width="0.3048" layer="3"/>
+<wire x1="-5" y1="27.75" x2="-0.25" y2="23" width="0.3048" layer="3"/>
+<via x="-0.25" y="23" extent="1-16" drill="0.35"/>
+<wire x1="-0.25" y1="23" x2="-0.75" y2="22.5" width="0.3048" layer="1"/>
+<wire x1="-0.75" y1="22.5" x2="-2.1" y2="22.5" width="0.3048" layer="1"/>
+<wire x1="-38.75" y1="27.75" x2="-5" y2="27.75" width="0.3048" layer="3"/>
+<via x="-0.31" y="22.46" extent="1-16" drill="0.35"/>
+<via x="8.07" y="14.63" extent="1-16" drill="0.35"/>
+<via x="2.42" y="11.61" extent="1-16" drill="0.35"/>
+<via x="-0.38" y="10.47" extent="1-16" drill="0.35"/>
+<via x="-39.36" y="28.98" extent="1-16" drill="0.35"/>
 <wire x1="23.13" y1="26.72" x2="23.1156" y2="26.5012" width="0" layer="19" extent="1-1"/>
 <wire x1="12.125" y1="26.875" x2="11.73" y2="26.83" width="0" layer="19" extent="1-1"/>
@@
 <wire x1="7.5" y1="14.48" x2="7.5" y2="14.48" width="0" layer="19" extent="1-3"/>
 <wire x1="3.875" y1="14.625" x2="3.87" y2="14.74" width="0" layer="19" extent="1-1"/>
+<wire x1="4" y1="14.5" x2="4.13" y2="14.48" width="0" layer="19" extent="1-1"/>
 <wire x1="4" y1="14.75" x2="3.87" y2="14.74" width="0" layer="19" extent="1-1"/>
-<wire x1="4" y1="14.5" x2="4.13" y2="14.48" width="0" layer="19" extent="1-1"/>
+<wire x1="-0.31" y1="22.46" x2="-0.75" y2="22.5" width="0" layer="19" extent="1-1"/>
+<wire x1="8.07" y1="14.63" x2="7.53" y2="14.51" width="0" layer="19" extent="1-3"/>
+<wire x1="2.42" y1="11.61" x2="2" y2="12" width="0" layer="19" extent="1-1"/>
+<wire x1="-39.36" y1="28.98" x2="-40" y2="29" width="0" layer="19" extent="1-1"/>
+<wire x1="-0.38" y1="10.47" x2="-1" y2="10.75" width="0" layer="19" extent="1-1"/>
+<wire x1="-19.405" y1="-23.185" x2="-19.405" y2="-23.925" width="0" layer="19" extent="1-1"/>
+<wire x1="4.595" y1="-23.185" x2="4.595" y2="-23.925" width="0" layer="19" extent="1-1"/>
+<wire x1="28.595" y1="-23.185" x2="28.595" y2="-23.925" width="0" layer="19" extent="1-1"/>
 <wire x1="23.22" y1="24.21" x2="23.1156" y2="26.5012" width="0" layer="19" extent="1-1"/>
 <wire x1="23.0958" y1="9.5176" x2="23.3" y2="13.35" width="0" layer="19" extent="1-1"/>
 <wire x1="22.89" y1="9.21" x2="23.0958" y2="9.5176" width="0" layer="19" extent="1-1"/>
 <wire x1="30.58736875" y1="9.08736875" x2="30.59" y2="9.08" width="0" layer="19" extent="1-1"/>
-<wire x1="-19.405" y1="-23.185" x2="-19.405" y2="-23.925" width="0" layer="19" extent="1-1"/>
-<wire x1="4.595" y1="-23.185" x2="4.595" y2="-23.925" width="0" layer="19" extent="1-1"/>
-<wire x1="28.595" y1="-23.185" x2="28.595" y2="-23.925" width="0" layer="19" extent="1-1"/>
 <wire x1="34.9624" y1="9.4668" x2="34.067" y2="9.5" width="0" layer="19" extent="1-1"/>
 </signal>
@@
 <signal name="N$39">
 <via x="10.47" y="28.03" extent="1-16" drill="0.35"/>
+<via x="10.73" y="27.42" extent="1-16" drill="0.35"/>
+<wire x1="10.73" y1="27.42" x2="10.47" y2="28.03" width="0" layer="19" extent="1-1"/>
 </signal>
 <signal name="DISABLE_PT2">
